Commit message: Session am Freitag weiter arbeiten an erstem Test.

File: gym_pybullet_drones/assets/target.urdf (robot description, URDF)
Before this commit: robot drone_target, 2 links, 1 joints
Links:
- link base_link: mass None -> 0

File: gym_pybullet_drones/assets/train_square.urdf (robot description, URDF)
Before this commit: robot drone_training_area, 6 links, 5 joints
Links:
- link base_link: mass None -> 0
