Commit message: - Dash App (Browser Dashboard) läuft nun - Dash App Ausgaben wurden auf Null umgeleitet, damit das Terminal nicht zugemüllt wird - Maze map_1.urdf Trägheitsdaten wurden ergänzt, um Fehlermeldungen zu verhindern - Anpassung der Kameraperspektive (Top-Down-View + Kamera immer über Drohne)

File: gym_pybullet_drones/assets/maze/map_1.urdf (robot description, URDF)
Before this commit: robot maze, 3 links, 2 joints
Links:
- link base_link: mass None -> 1
- link walls: mass None -> 10
