Commit message: - Neue Datei zur Erstellung der URDF Dateien - Hinzufügen neuer maze urdfs

File: gym_pybullet_drones/assets/maze/map_0.urdf (robot description, URDF)
Before this commit: robot maze, 3 links, 2 joints
Links:
- link walls: mass 343 -> 355; geometry collision box size=0.05 0.05 1; collision box size=0.05 0.05 1

File: gym_pybullet_drones/assets/maze/map_1.urdf (robot description, URDF)
Before this commit: robot maze, 3 links, 2 joints
Links:
- link walls: mass 10 -> 377

File: gym_pybullet_drones/assets/maze/map_10.urdf (robot description, URDF)
Before this commit: robot maze, 3 links, 2 joints
Links:
- link base_link: mass None -> 1
- link walls: mass None -> 374

File: gym_pybullet_drones/assets/maze/map_11.urdf (robot description, URDF)
Before this commit: robot maze, 3 links, 2 joints
Links:
- link base_link: mass None -> 1
- link walls: mass None -> 363

File: gym_pybullet_drones/assets/maze/map_12.urdf (robot description, URDF)
Before this commit: robot maze, 3 links, 2 joints
Links:
- link base_link: mass None -> 1
- link walls: mass None -> 370

File: gym_pybullet_drones/assets/maze/map_13.urdf (robot description, URDF)
Before this commit: robot maze, 3 links, 2 joints
Links:
- link base_link: mass None -> 1
- link walls: mass None -> 389

File: gym_pybullet_drones/assets/maze/map_14.urdf (robot description, URDF)
Before this commit: robot maze, 3 links, 2 joints
Links:
- link base_link: mass None -> 1
- link walls: mass None -> 432

File: gym_pybullet_drones/assets/maze/map_15.urdf (robot description, URDF)
Before this commit: robot maze, 3 links, 2 joints
Links:
- link base_link: mass None -> 1
- link walls: mass None -> 428

File: gym_pybullet_drones/assets/maze/map_16.urdf (robot description, URDF)
Before this commit: robot maze, 3 links, 2 joints
Links:
- link base_link: mass None -> 1
- link walls: mass None -> 491

File: gym_pybullet_drones/assets/maze/map_17.urdf (robot description, URDF)
Before this commit: robot maze, 3 links, 2 joints
Links:
- link base_link: mass None -> 1
- link walls: mass None -> 516

File: gym_pybullet_drones/assets/maze/map_18.urdf (robot description, URDF)
Before this commit: robot maze, 3 links, 2 joints
Links:
- link base_link: mass None -> 1
- link walls: mass None -> 447

File: gym_pybullet_drones/assets/maze/map_19.urdf (robot description, URDF)
Before this commit: robot maze, 3 links, 2 joints
Links:
- link base_link: mass None -> 1
- link walls: mass None -> 462

File: gym_pybullet_drones/assets/maze/map_2.urdf (robot description, URDF)
Before this commit: robot maze, 3 links, 2 joints
Links:
- link base_link: mass None -> 1
- link walls: mass None -> 378

File: gym_pybullet_drones/assets/maze/map_20.urdf (robot description, URDF)
Before this commit: robot maze, 3 links, 2 joints
Links:
- link base_link: mass None -> 1
- link walls: mass None -> 466

File: gym_pybullet_drones/assets/maze/map_3.urdf (robot description, URDF)
Before this commit: robot maze, 3 links, 2 joints
Links:
- link base_link: mass None -> 1
- link walls: mass None -> 388

File: gym_pybullet_drones/assets/maze/map_5.urdf (robot description, URDF)
Before this commit: robot maze, 3 links, 2 joints
Links:
- link base_link: mass None -> 1
- link walls: mass None -> 323

File: gym_pybullet_drones/assets/maze/map_6.urdf (robot description, URDF)
Before this commit: robot maze, 3 links, 2 joints
Links:
- link base_link: mass None -> 1
- link walls: mass None -> 366

File: gym_pybullet_drones/assets/maze/map_7.urdf (robot description, URDF)
Before this commit: robot maze, 3 links, 2 joints
Links:
- link base_link: mass None -> 1
- link walls: mass None -> 370

File: gym_pybullet_drones/assets/maze/map_8.urdf (robot description, URDF)
Before this commit: robot maze, 3 links, 2 joints
Links:
- link base_link: mass None -> 1
- link walls: mass None -> 371

File: gym_pybullet_drones/assets/maze/map_9.urdf (robot description, URDF)
Before this commit: robot maze, 3 links, 2 joints
Links:
- link base_link: mass None -> 1
- link walls: mass None -> 348
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