Commit message: Fixed new Maze URDFs, Fixed the order and random selection of mazes/starting positions, change standard safe to all 50.000 iterations

File: gym_pybullet_drones/assets/maze/map_27.urdf (robot description, URDF)
Before this commit: robot maze, 3 links, 2 joints
Links:
- link base_link: mass None -> 1
- link walls: mass None -> 1

File: gym_pybullet_drones/assets/maze/map_28.urdf (robot description, URDF)
Before this commit: robot maze, 3 links, 2 joints
Links:
- link base_link: mass None -> 1
- link walls: mass None -> 1

File: gym_pybullet_drones/assets/maze/map_29.urdf (robot description, URDF)
Before this commit: robot maze, 3 links, 2 joints
Links:
- link base_link: mass None -> 1
- link walls: mass None -> 1

File: gym_pybullet_drones/assets/maze/map_30.urdf (robot description, URDF)
Before this commit: robot maze, 3 links, 2 joints
Links:
- link base_link: mass None -> 1
- link walls: mass None -> 1

File: gym_pybullet_drones/assets/maze/map_31.urdf (robot description, URDF)
Before this commit: robot maze, 3 links, 2 joints
Links:
- link base_link: mass None -> 1
- link walls: mass None -> 1
